File: a5e_kicad/hyperbus.kicad_sch (KiCad schematic)
At the start: 4 parts, among them U1901 Ram x8

Commit message: add vias to lppdr balls
Parts:
- renumbered C1901 to C97, C1902 to C98, C1903 to C99, U1901 to U13
Changed lines of the file:
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@@
 		(in_pos_files yes)
 		(dnp no)
-		(property "Reference" "U1901"
+		(property "Reference" "U13"
 			(at 109.22 38.1 0)
 			(show_name no)
@@
 			(project "agilex_3_soc"
 				(path "/a5b98d95-6877-4284-904f-d04e32723ae0/a8f2fee3-4477-4348-8890-5a8bd0c95ceb"
-					(reference "U1901")
+					(reference "U13")
 					(unit 1)
 				)
@@
 		(dnp no)
 		(fields_autoplaced yes)
-		(property "Reference" "#PWR01903"
+		(property "Reference" "#PWR0115"
 			(at 181.61 40.64 0)
 			(hide yes)
@@
 			(project "agilex_3_soc"
 				(path "/a5b98d95-6877-4284-904f-d04e32723ae0/a8f2fee3-4477-4348-8890-5a8bd0c95ceb"
-					(reference "#PWR01903")
+					(reference "#PWR0115")
 					(unit 1)
 				)
@@
 		(in_pos_files yes)
 		(dnp no)
-		(property "Reference" "#PWR01901"
+		(property "Reference" "#PWR0113"
 			(at 144.78 90.17 0)
 			(hide yes)
@@
 			(project "agilex_3_soc"
 				(path "/a5b98d95-6877-4284-904f-d04e32723ae0/a8f2fee3-4477-4348-8890-5a8bd0c95ceb"
-					(reference "#PWR01901")
+					(reference "#PWR0113")
 					(unit 1)
 				)
@@
 		(in_pos_files yes)
 		(dnp no)
-		(property "Reference" "C1903"
+		(property "Reference" "C99"
 			(at 182.88 46.99 0)
 			(show_name no)
@@
 			(project "agilex_3_soc"
 				(path "/a5b98d95-6877-4284-904f-d04e32723ae0/a8f2fee3-4477-4348-8890-5a8bd0c95ceb"
-					(reference "C1903")
+					(reference "C99")
 					(unit 1)
 				)
@@
 		(in_pos_files yes)
 		(dnp no)
-		(property "Reference" "#PWR01902"
+		(property "Reference" "#PWR0114"
 			(at 175.26 62.23 0)
 			(hide yes)
@@
 			(project "agilex_3_soc"
 				(path "/a5b98d95-6877-4284-904f-d04e32723ae0/a8f2fee3-4477-4348-8890-5a8bd0c95ceb"
-					(reference "#PWR01902")
+					(reference "#PWR0114")
 					(unit 1)
 				)
@@
 		(in_pos_files yes)
 		(dnp no)
-		(property "Reference" "C1902"
+		(property "Reference" "C98"
 			(at 175.26 46.99 0)
 			(show_name no)
@@
 			(project "agilex_3_soc"
 				(path "/a5b98d95-6877-4284-904f-d04e32723ae0/a8f2fee3-4477-4348-8890-5a8bd0c95ceb"
-					(reference "C1902")
+					(reference "C98")
 					(unit 1)
 				)
@@
 		(dnp no)
 		(fields_autoplaced yes)
-		(property "Reference" "#PWR01904"
+		(property "Reference" "#PWR0116"
 			(at 181.61 43.18 0)
 			(hide yes)
@@
 			(project "agilex_3_soc"
 				(path "/a5b98d95-6877-4284-904f-d04e32723ae0/a8f2fee3-4477-4348-8890-5a8bd0c95ceb"
-					(reference "#PWR01904")
+					(reference "#PWR0116")
 					(unit 1)
 				)
@@
 		(in_pos_files yes)
 		(dnp no)
-		(property "Reference" "C1901"
+		(property "Reference" "C97"
 			(at 167.64 46.99 0)
 			(show_name no)
@@
 			(project "agilex_3_soc"
 				(path "/a5b98d95-6877-4284-904f-d04e32723ae0/a8f2fee3-4477-4348-8890-5a8bd0c95ceb"
-					(reference "C1901")
-					(unit 1)
-				)
+					(reference "C97")
+					(unit 1)
+				)
