File: a5e_kicad/ps.kicad_sch (KiCad schematic)
At the start: 48 parts

Commit message: fix clock routing and move all components inside board perimeters
Parts:
- U15: value (none) -> TDA38812XUMA1
Changed lines of the file:
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@@
 			)
 		)
-		(property "Value" ""
+		(property "Value" "TDA38812XUMA1"
 			(at 153.67 90.17 0)
 			(show_name no)

Commit message: start finishing the pcb
Changed lines of the file:
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@@
 		(in_pos_files yes)
 		(dnp no)
-		(fields_autoplaced yes)
 		(property "Reference" "U15"
 			(at 159.6233 54.61 0)
@@
 		)
 		(property "Value" "TDA38812XUMA1"
-			(at 153.67 90.17 0)
+			(at 152.908 87.122 0)
 			(show_name no)
 			(do_not_autoplace no)
