File: a5e_kicad/clk.kicad_sch (KiCad schematic)
At the start: 11 parts, among them Y2 ASV-xxxMHz

Commit message: choose clock ic:s
Parts:
- U9: value (none) -> AX3HAF1-100.0000; footprint agilex_lib:XL7 -> agilex_lib:AX3_3225_6Pin_3.2x2.5mm; symbol agilex_5_lib:XLL7 -> agilex_5_lib:AX3HAF1-100.0000
- Y2: value ASV-xxxMHz -> SIT8924BA-73-18N-25.000000; footprint Oscillator:Oscillator_SMD_Abracon_ASV-4Pin_7.0x5.1mm -> agilex_lib:SIT8924_2520_4Pin_2.5x2.0mm; symbol Oscillator:ASV-xxxMHz -> agilex_5_lib:SIT8924BA-73-18N-25.000000
Connections:
- net 1V8: no longer Y2.4 (Vdd)
- net 3v3: no longer U9.6 (Vcc)
- net GND: no longer U9.3 (GND), Y2.2 (GND)
- net clk1_P: no longer Y2.3 (OUT)
- net at R26.1: no longer U9.5 (OUT-)
- net at R50.2: no longer Y2.1 (EN)
- net at R25.1: no longer U9.4 (OUT+)
Changed lines of the file:
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@@
 	)
 	(symbol
-		(lib_id "Oscillator:ASV-xxxMHz")
+		(lib_id "agilex_5_lib:SIT8924BA-73-18N-25.000000")
 		(at 107.95 109.22 0)
 		(unit 1)
@@
 			)
 		)
-		(property "Value" "ASV-xxxMHz"
+		(property "Value" "SIT8924BA-73-18N-25.000000"
 			(at 120.65 105.3398 0)
 			(show_name no)
@@
 			)
 		)
-		(property "Footprint" "Oscillator:Oscillator_SMD_Abracon_ASV-4Pin_7.0x5.1mm"
+		(property "Footprint" "agilex_lib:SIT8924_2520_4Pin_2.5x2.0mm"
 			(at 125.73 118.11 0)
-			(hide yes)
-			(show_name no)
-			(do_not_autoplace no)
-			(effects
-				(font
-					(size 1.27 1.27)
-				)
-			)
-		)
-		(property "Datasheet" "http://www.abracon.com/Oscillators/ASV.pdf"
+			(show_name no)
+			(do_not_autoplace no)
+			(hide yes)
+			(effects
+				(font
+					(size 1.27 1.27)
+				)
+			)
+		)
+		(property "Datasheet" "https://www.mouser.com/datasheet/2/371/SiT8924-datasheet-1839508.pdf"
 			(at 105.41 109.22 0)
-			(hide yes)
-			(show_name no)
-			(do_not_autoplace no)
-			(effects
-				(font
-					(size 1.27 1.27)
-				)
-			)
-		)
-		(property "Description" "3.3V HCMOS SMD Crystal Clock Oscillator, Abracon"
+			(show_name no)
+			(do_not_autoplace no)
+			(hide yes)
+			(effects
+				(font
+					(size 1.27 1.27)
+				)
+			)
+		)
+		(property "Description" "25MHz 1.8V LVCMOS XO, SiTime MEMS, NC pin1 (always enabled)"
 			(at 107.95 109.22 0)
-			(hide yes)
-			(show_name no)
-			(do_not_autoplace no)
+			(show_name no)
+			(do_not_autoplace no)
+			(hide yes)
 			(effects
 				(font
@@
 		(pin "1"
 		)
+		(pin "2"
+		)
 		(pin "3"
 		)
 		(pin "4"
-		)
-		(pin "2"
 		)
 		(instances
@@
 	)
 	(symbol
-		(lib_id "agilex_5_lib:XLL7")
+		(lib_id "agilex_5_lib:AX3HAF1-100.0000")
 		(at 95.25 57.15 0)
 		(unit 1)
@@
 					(size 1.27 1.27)
 				)
-				(justify left)
-			)
-		)
-		(property "Value" ""
+			)
+		)
+		(property "Value" "AX3HAF1-100.0000"
 			(at 95.25 57.15 0)
 			(show_name no)
@@
 			)
 		)
-		(property "Footprint" "agilex_lib:XL7"
+		(property "Footprint" "agilex_lib:AX3_3225_6Pin_3.2x2.5mm"
 			(at 95.25 57.15 0)
-			(hide yes)
-			(show_name no)
-			(do_not_autoplace no)
-			(effects
-				(font
-					(size 1.27 1.27)
-				)
-			)
-		)
-		(property "Datasheet" ""
+			(show_name no)
+			(do_not_autoplace no)
+			(hide yes)
+			(effects
+				(font
+					(size 1.27 1.27)
+				)
+			)
+		)
+		(property "Datasheet" "https://abracon.com/datasheets/AX3.pdf"
 			(at 95.25 57.15 0)
-			(hide yes)
-			(show_name no)
-			(do_not_autoplace no)
-			(effects
-				(font
-					(size 1.27 1.27)
-				)
-			)
-		)
-		(property "Description" ""
+			(show_name no)
+			(do_not_autoplace no)
+			(hide yes)
+			(effects
+				(font
+					(size 1.27 1.27)
+				)
+			)
+		)
+		(property "Description" "100MHz HCSL differential XO, 3.3V, Abracon ClearClock AX3"
 			(at 95.25 57.15 0)
-			(hide yes)
-			(show_name no)
-			(do_not_autoplace no)
-			(effects
-				(font
-					(size 1.27 1.27)
-				)
-			)
+			(show_name no)
+			(do_not_autoplace no)
+			(hide yes)
+			(effects
+				(font
+					(size 1.27 1.27)
+				)
+			)
+		)
+		(pin "1"
+		)
+		(pin "2"
+		)
+		(pin "3"
 		)
 		(pin "4"
@@
 		)
 		(pin "6"
-		)
-		(pin "2"
-		)
-		(pin "3"
-		)
-		(pin "1"
 		)
 		(instances
@@
 		)
 	)
+	(wire
+		(pts
+			(xy 83.82 59.69) (xy 83.82 48.26)
+		)
+		(stroke
+			(width 0)
+			(type default)
+		)
+	)
+	(wire
+		(pts
+			(xy 83.82 48.26) (xy 95.25 48.26)
+		)
+		(stroke
+			(width 0)
+			(type default)
+		)
+	)
+	(junction
+		(at 95.25 48.26)
+		(diameter 0)
+		(color 0 0 0 0)
+	)
 )
