File: a5e_kicad/fpga_power.kicad_sch (KiCad schematic)
At the start: 2 parts, among them U7 A5EB013B-B23B

Commit message: update project
Connections:
- net 1V2: now also U7.CW57 (VCCIO_PIO_SDM)
- net 1V8: no longer U7.CT54 (VCC_IO_SDM), U7.CW57 (VCCIO_PIO_SDM)
- net VCORE: now also U7.CT54 (VCC_IO_SDM)
Changed lines of the file:
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@@
 			)
 		)
-		(property "Value" "1V8"
+		(property "Value" "VCORE"
 			(at 153.67 121.9199 90)
 			(show_name no)
@@
 			)
 		)
-		(property "Value" "1V8"
+		(property "Value" "1V2"
 			(at 128.27 96.5199 90)
 			(show_name no)
