File: a5e_kicad/fpga_power.kicad_sch (KiCad schematic)
At the start: 2 parts, among them U7 A5EB013B-B23B

Commit message: Rename lowercase 3v3/1v8 power symbols to 3V3/1V8
KiCad already merged them into the same nets, but every mixed-case pair
raised a similar_power ERC warning. No connectivity change. ERC 503 -> 339.
Connections:
- net 3v3 renamed 3V3
Changed lines of the file:
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@@
 			)
 		)
-		(property "Value" "3v3"
+		(property "Value" "3V3"
 			(at 49.53 147.3199 90)
 			(show_name no)
@@
 			)
 		)
-		(property "Value" "3v3"
+		(property "Value" "3V3"
 			(at 125.73 50.7999 90)
 			(show_name no)
@@
 			)
 		)
-		(property "Value" "3v3"
+		(property "Value" "3V3"
 			(at 135.89 27.9399 90)
 			(show_name no)
@@
 			)
 		)
-		(property "Value" "3v3"
+		(property "Value" "3V3"
 			(at 49.53 139.6999 90)
 			(show_name no)
