File: a5e_kicad/fpga_power.kicad_sch (KiCad schematic)
At the start: 2 parts, among them U7 A5EB013B-B23B

Commit message: Add LCSC part numbers and fix C102 footprint
Add a hidden LCSC field to 290 symbols from the JLCPCB parts match
(2026-10-23). Left without LCSC: U7, U15, L1 (not in the JLCPCB
library), C1/C2/C4 and L2-L5 (no value specified), J3 (no confident
match) and Y3 (the 12 pF Basic crystal does not suit the 27 pF load
caps). U2, U12, Y2 and J9 carry the exact-MPN LCSC numbers although
they currently show zero JLCPCB stock.

C102 (22U 6V3) had a 0201 footprint; no 22 uF 0201 part exists. Change
it to 0402 (C415703) like C5-C7.
Parts:
- C102: footprint Capacitor_SMD:C_0201_0603Metric -> Capacitor_SMD:C_0402_1005Metric; LCSC (none) -> C415703
Changed lines of the file:
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@@
 			)
 		)
-		(property "Footprint" "Capacitor_SMD:C_0201_0603Metric"
+		(property "Footprint" "Capacitor_SMD:C_0402_1005Metric"
 			(at 44.1452 156.21 0)
 			(hide yes)
+			(show_name no)
+			(do_not_autoplace no)
+			(effects
+				(font
+					(size 1.27 1.27)
+				)
+			)
+		)
+		(property "LCSC" "C415703"
+			(at 44.1452 156.21 0)
+			(hide yes)

Commit message: Power/config review against the Altera docs: bank 6A, MSEL, resets, fabric clock
Checked against Pin Connection Guidelines 813266, Power Management UG
813161, Configuration UG 813773 and the data sheet 813918; findings are
in AGILEX_POWER_CONFIG_CHECKLIST.md.

- VCCIO_HVIO_6A moves from the VCCPT 1V8 regulator to 3V3. PCG table 32
  requires a dedicated VCCIO_HVIO supply. CE19 no longer takes the 1.8 V
  sdm_clk25.
- Y4 (YXC OT3225100MJBA4SL, 100 MHz 3.3 V CMOS, C4353707) drives the
  dangling clk100 net to AE11 (bank 6G PLLREFCLK1), giving the fabric a
  PLL reference that doesn't depend on the HPS. The clock sheet pin
  clk2_N is renamed clk100.
- MSEL 001 (AS fast) -> 011 (AS normal): fast mode needs all supplies
  ramped within 10 ms, which the sequenced regulators don't guarantee.
  R45 now goes to 1V8, and R4 gets its own GND.
- R264 10k pull-up on HPS_COLD_nRESET (SDM_IO10), as the PCG requires.
- R9/R10 (INIT_DONE/CONF_DONE pull-ups) DNP; the internal pull-downs
  hold the pins low until configuration.
- Note on the fpga_power sheet and the PCB (Cmts.User): ferrite + cap
  isolation filters on the PLL/ADC rails are recommended but not
  fitted yet.
Connections:
- net 1V8: no longer U7.CL29 (VCCIO_HVIO_6A), U7.CT29 (VCCIO_HVIO_6A)
- net 3V3: now also U7.CL29 (VCCIO_HVIO_6A), U7.CT29 (VCCIO_HVIO_6A)
Other:
- note added: "6A bank at 3.3 V like 6B-6H (VCCIO_HVIO needs a dedicated supply, PCG table 32); fabric PLL refclk = Y4 100 MHz on AE11 (bank 6G)"
- note added: "RECOMMENDED (not fitted yet): isolation filters per PCG 813266 table 32 - ferrite bead (e.g. BLM15PX121SN1) + 4.7u || 100n at each pin group: 1V8: VCCPLL1_HPS, VCCPLL2_HPS, VCCADC, VCCPLL_SDM VCORE: VCCPLLDIG1_HPS, VCCPLLDIG2_HPS, VCCPLLDIG_SDM"
- note removed: "6A bank at 1.8 V: 25 MHz refclk on CE19"
Changed lines of the file:
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@@
 		(rev "0.1")
 	)
-	(text "6A bank at 1.8 V: 25 MHz refclk on CE19"
+	(text "6A bank at 3.3 V like 6B-6H (VCCIO_HVIO needs a dedicated supply, PCG table 32);\nfabric PLL refclk = Y4 100 MHz on AE11 (bank 6G)"
 		(exclude_from_sim no)
 		(at 52.832 159.512 0)
@@
 			)
 		)
-		(property "Value" "1V8"
+		(property "Value" "3V3"
 			(at 49.53 132.0799 90)
 			(show_name no)
@@
 		)
 	)
+	(text "RECOMMENDED (not fitted yet): isolation filters per PCG 813266 table 32 -\nferrite bead (e.g. BLM15PX121SN1) + 4.7u || 100n at each pin group:\n1V8: VCCPLL1_HPS, VCCPLL2_HPS, VCCADC, VCCPLL_SDM\nVCORE: VCCPLLDIG1_HPS, VCCPLLDIG2_HPS, VCCPLLDIG_SDM"
+		(exclude_from_sim no)
+		(at 52.832 172.72 0)
+		(effects
+			(font
+				(size 1.27 1.27)
+			)
+			(justify left)
+		)
+	)

Commit message: Schematic reorg step 1: remove dangling stubs and stale notes, correct notes, fill title blocks
Netlist: 0 renamed, 0 connectivity diffs; DRC parity 0. ERC 315 -> 242.
Plan refreshed for the eMMC, RTL8211FDI, TPS548A28 and the tuned LPDDR4 (IOBANK 3 sheet name kept).
Other:
- title: (none) -> SoC power pins
Changed lines of the file:
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@@
 	(paper "A4")
 	(title_block
-		(rev "0.1")
+		(title "SoC power pins")
+		(rev "${REVISION}")
+		(comment 1 "${BOARD}")
 	)
 	(text "RECOMMENDED (not fitted yet): isolation filters per PCG 813266 table 32 -\nferrite bead (e.g. BLM15PX121SN1) + 4.7u || 100n at each pin group:\n1V8: VCCPLL1_HPS, VCCPLL2_HPS, VCCADC, VCCPLL_SDM\nVCORE: VCCPLLDIG1_HPS, VCCPLLDIG2_HPS, VCCPLLDIG_SDM"
@@
 	)
 	(junction
-		(at 43.18 119.38)
-		(diameter 0)
-		(color 0 0 0 0)
-	)
-	(junction
 		(at 162.56 38.1)
 		(diameter 0)
@@
 		(pts
 			(xy 254 31.75) (xy 254 29.21)
-		)
-		(stroke
-			(width 0)
-			(type default)
-		)
-	)
-	(wire
-		(pts
-			(xy 30.48 119.38) (xy 43.18 119.38)
 		)
 		(stroke
@@
 		(effects
 			(font
-				(size 1.27 1.27)
-			)
-			(justify right)
-		)
-	)
-	(hierarchical_label "1v8"
-		(shape output)
-		(at 30.48 119.38 180)
-		(effects
-			(font
