File: a5e_kicad/fpga_gnd.kicad_sch (KiCad schematic)
At the start: 1 part, among them U7 A5EB013B-B23B

Commit message: U7: use Altera_B23B footprint from Rolf-Altera's generator
Generated with the KiCad footprint generator from Rolf-Altera's
kicad-library-tools branch Altera_Agilex_5 (4024449, MR
kicad/libraries/kicad-library-tools!2200), which uses Altera's
B23B ball coordinate / land pattern file (PBC-LPG):
  py generate.py -g package/grid_array -p Altera_B23B

- Pads per Altera land pattern: 0.305 mm (769), 0.33 mm (17),
  0.355 mm (9), NSMD with mask = pad + 0.1 mm. Old footprint had
  0.4 mm pads with 0.075 mm clearance overrides and a duplicated
  CL23 pad.
- Placed at rotation 0 on the package centre (156.4668, 112.1692);
  every ball lands exactly on its old position (max deviation
  0.0000 mm), so routing is unchanged. The old footprint origin was
  0.1 mm off the package centre, which would have offset assembly.
- Nets carried over by ball number; schematic footprint field updated.

DRC clearance errors 101 -> 16 (U7 BGA escape now meets JLCPCB 0.09 mm).
New: 5 courtyard overlaps (R24, R252-R255) with the KLC 1 mm BGA
courtyard; the parts are 0.27-0.49 mm outside the package body.

Co-Authored-By: Claude Opus 5.5 <noreply@anthropic.com>
Parts:
- U7: footprint agilex_lib:VFBGA_b23b_mirror -> agilex_lib:Altera_B23B
Changed lines of the file:
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@@
 			)
 		)
-		(property "Footprint" "agilex_lib:VFBGA_b23b_mirror"
+		(property "Footprint" "agilex_lib:Altera_B23B"
 			(at 213.36 63.5 0)
 			(hide yes)
@@
 			)
 		)
-		(property "Footprint" "agilex_lib:VFBGA_b23b_mirror"
+		(property "Footprint" "agilex_lib:Altera_B23B"
 			(at 55.88 83.82 0)
 			(hide yes)
@@
 			)
 		)
-		(property "Footprint" "agilex_lib:VFBGA_b23b_mirror"
+		(property "Footprint" "agilex_lib:Altera_B23B"
 			(at 129.54 83.82 0)
 			(hide yes)
