File: a5e_kicad/fpga_gnd.kicad_sch (KiCad schematic)
At the start: 1 part, among them U7 A5EB013B-B23B

Commit message: Schematic reorg step 1: remove dangling stubs and stale notes, correct notes, fill title blocks
Netlist: 0 renamed, 0 connectivity diffs; DRC parity 0. ERC 315 -> 242.
Plan refreshed for the eMMC, RTL8211FDI, TPS548A28 and the tuned LPDDR4 (IOBANK 3 sheet name kept).
Other:
- title: (none) -> SoC ground pins
Changed lines of the file:
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@@
 	(paper "A4")
 	(title_block
-		(rev "0.1")
+		(title "SoC ground pins")
+		(rev "${REVISION}")
+		(comment 1 "${BOARD}")
 	)
 	(junction
