File: a5e_kicad/clocks.kicad_sch (KiCad schematic)
At the start: 18 parts, among them U9 AX3DAF1-100.0000T, Y2 SIT8924BA-78-18E-25.000000, Y4 OT3225100MJBA4SL 100MHz

Commit message: Ethernet PHY passives to 0201, R27/R28 to 0402, preliminary RGMII routing
- 31 PHY passives on the hps_ethernet sheet 0402 -> 0201 (C24 22u stays
  0402): 100n C190183, 1u C272877, 27p C85899, 10k C473048,
  330R C516485, 4K7 C270346, 1K5 C270361, 2K49 C473476.
- Refclk bias R27/R28 0201 -> 0402 (C25120, 49.9R); R28 moved 0.1 mm
  to +x to clear the refclk_N meander.
- Preliminary RGMII routing: RX on F.Cu, TX on In2. Group spread
  TX 79 ps (TXD1 longest), RX 44 ps.
- Schematic sheets as saved by eeschema.
Parts:
- R27, R28: footprint Resistor_SMD:R_0201_0603Metric -> Resistor_SMD:R_0402_1005Metric; LCSC C170197 -> C25120
Changed lines of the file:
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@@
 			)
 		)
-		(property "Footprint" "Resistor_SMD:R_0201_0603Metric"
+		(property "Footprint" "Resistor_SMD:R_0402_1005Metric"
 			(at 149.098 67.31 90)
 			(hide yes)
@@
 			)
 		)
-		(property "LCSC" "C170197"
+		(property "LCSC" "C25120"
 			(at 149.098 67.31 90)
 			(hide yes)
@@
 			)
 		)
-		(property "Footprint" "Resistor_SMD:R_0201_0603Metric"
+		(property "Footprint" "Resistor_SMD:R_0402_1005Metric"
 			(at 157.988 67.31 90)
 			(hide yes)
@@
 			)
 		)
-		(property "LCSC" "C170197"
+		(property "LCSC" "C25120"
 			(at 157.988 67.31 90)
 			(hide yes)
