File: a5e_kicad/debug_status.kicad_sch (KiCad schematic)
At the start: 13 parts, among them J1 Conn_01x05, J10 HPS_UART_3V3, J2 Conn_01x03, U1 SN74AXC4T774PWR, U42 SN74AXC4T774PWR

Commit message: Schematic reorg step 7: no global labels, NC flags on unused U7 pins
- hps_uart0_tx/rx, eth_rst_n, phy_rst_n, fpga_led: global labels replaced by
  sheet pins; eth_led_g_n is a local label
- HyperBus labels/bus, the HPS {hps_i2c} bus and the pwr_scl/pwr_sda wiring
  removed (nothing behind them)
- 118 U7 pins that only had a net label: label, stub and bus entry removed,
  no-connect flag added
- Bank 3A notes restacked
- PCB: 124 nets renamed (118 to unconnected-(U7...))

Netdiff: 124 renamed, 0 connectivity diffs. ERC 148 -> 21. DRC parity 0.
Changed lines of the file:
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@@
 		)
 	)
-	(global_label "hps_uart0_rx"
+	(hierarchical_label "hps_uart0_rx"
 		(shape output)
 		(at 21.59 147.32 180)
@@
 			(justify right)
 		)
-		(property "Intersheetrefs" "${INTERSHEET_REFS}"
-			(at 21.59 147.32 0)
-			(hide yes)
-			(show_name no)
-			(do_not_autoplace no)
-			(effects
-				(font
-					(size 1.27 1.27)
-				)
-			)
-		)
 	)
-	(global_label "eth_rst_n"
+	(hierarchical_label "eth_rst_n"
 		(shape input)
 		(at 21.59 149.86 180)
@@
 			(justify right)
 		)
-		(property "Intersheetrefs" "${INTERSHEET_REFS}"
-			(at 21.59 149.86 0)
-			(hide yes)
-			(show_name no)
-			(do_not_autoplace no)
-			(effects
-				(font
-					(size 1.27 1.27)
-				)
-			)
-		)
 	)
 	(hierarchical_label "fpga_uart_tx"
@@
 		)
 	)
-	(global_label "phy_rst_n"
+	(hierarchical_label "phy_rst_n"
 		(shape output)
 		(at 68.58 149.86 0)
@@
 			(justify left)
 		)
-		(property "Intersheetrefs" "${INTERSHEET_REFS}"
-			(at 68.58 149.86 0)
-			(hide yes)
-			(show_name no)
-			(do_not_autoplace no)
-			(effects
-				(font
-					(size 1.27 1.27)
-				)
-			)
-		)
 	)
 	(label "pg_all_3v3"
@@
 		)
 	)
-	(global_label "hps_uart0_tx"
+	(hierarchical_label "hps_uart0_tx"
 		(shape input)
 		(at 21.59 144.78 180)
@@
 			(justify right)
 		)
-		(property "Intersheetrefs" "${INTERSHEET_REFS}"
-			(at 21.59 144.78 0)
-			(hide yes)
-			(show_name no)
-			(do_not_autoplace no)
-			(effects
-				(font
-					(size 1.27 1.27)
-				)
-			)
-		)
 	)
 	(symbol
@@
 		)
 	)
-	(global_label "fpga_led"
+	(hierarchical_label "fpga_led"
 		(shape input)
 		(at 181.61 78.74 0)
@@
 			(justify left)
 		)
-		(property "Intersheetrefs" "${INTERSHEET_REFS}"
-			(at 181.61 78.74 0)
-			(hide yes)
-			(show_name no)
-			(do_not_autoplace no)
-			(effects
-				(font
-					(size 1.27 1.27)
-				)
-			)
-		)
 	)
