File: a5e_kicad/io_headers.kicad_sch (KiCad schematic)
At the start: 9 parts, among them J3 2x19 1.27mm socket, bottom, J5 Conn_01x14

Commit message: Schematic reorg step 9: ERC to zero
- Wires trimmed back to their last label or cap (SDM config lines, LPDDR4
  decoupling rows, PG pins); loose stubs and R29 leftovers removed
- Unused bus links removed: {iob6a}, {iobank_2aB}, {iob6c}, {phy} and the
  io_headers {jtag} (sheet pins, root buses, unnamed internal buses);
  {iob6b} bus tail trimmed

Netdiff: 0 renamed, 0 connectivity diffs. ERC 21 -> 0. PCB unchanged, DRC parity 0.
Changed lines of the file:
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@@
 		(comment 1 "${BOARD}")
-	)
-	(junction
-		(at 35.56 134.62)
-		(diameter 0)
-		(color 0 0 0 0)
-	)
-	(bus
-		(pts
-			(xy 284.48 27.94) (xy 284.48 129.54)
-		)
-		(stroke
-			(width 0)
-			(type default)
-		)
-	)
-	(bus
-		(pts
-			(xy 30.48 134.62) (xy 35.56 134.62)
-		)
-		(stroke
-			(width 0)
-			(type default)
-		)
-	)
-	(bus
-		(pts
-			(xy 35.56 193.04) (xy 116.84 193.04)
-		)
-		(stroke
-			(width 0)
-			(type default)
-		)
-	)
-	(bus
-		(pts
-			(xy 35.56 134.62) (xy 35.56 193.04)
-		)
-		(stroke
-			(width 0)
-			(type default)
-		)
-	)
-	(bus
-		(pts
-			(xy 264.16 134.62) (xy 276.86 134.62)
-		)
-		(stroke
-			(width 0)
-			(type default)
-		)
-	)
-	(bus
-		(pts
-			(xy 35.56 134.62) (xy 119.38 134.62)
-		)
-		(stroke
-			(width 0)
-			(type default)
-		)
-	)
-	(bus
-		(pts
-			(xy 241.3 129.54) (xy 284.48 129.54)
-		)
-		(stroke
-			(width 0)
-			(type default)
-		)
 	)
 	(bus
@@
 			(width 0)
 			(type default)
-		)
-	)
-	(bus
-		(pts
-			(xy 30.48 116.84) (xy 68.58 116.84)
-		)
-		(stroke
-			(width 0)
-			(type default)
-		)
-	)
-	(label "{jtag}"
-		(at 264.16 134.62 0)
-		(effects
-			(font
-				(size 1.27 1.27)
-			)
-			(justify left bottom)
 		)
 	)
@@
 		)
 	)
-	(hierarchical_label "{iob6c}"
-		(shape bidirectional)
-		(at 27.94 121.92 180)
-		(effects
-			(font
-				(size 1.27 1.27)
-			)
-			(justify right)
-		)
-	)
-	(hierarchical_label "{phy}"
-		(shape bidirectional)
-		(at 30.48 116.84 180)
-		(effects
-			(font
-				(size 1.27 1.27)
-			)
-			(justify right)
-		)
-	)
-	(hierarchical_label "{iobank_2aB}"
-		(shape bidirectional)
-		(at 30.48 134.62 180)
-		(effects
-			(font
-				(size 1.27 1.27)
-			)
-			(justify right)
-		)
-	)
 	(hierarchical_label "{iob6h}"
 		(shape bidirectional)
 		(at 27.94 132.08 180)
-		(effects
-			(font
-				(size 1.27 1.27)
-			)
-			(justify right)
-		)
-	)
-	(hierarchical_label "{jtag}"
-		(shape bidirectional)
-		(at 264.16 134.62 180)
 		(effects
 			(font
@@
 		(effects
 			(font
-				(size 1.27 1.27)
-			)
-			(justify right)
-		)
-	)
-	(hierarchical_label "{iob6a}"
-		(shape bidirectional)
-		(at 27.94 119.38 180)
-		(effects
-			(font
