File: a5e_kicad/pwr_rails.kicad_sch (KiCad schematic)
At the start: 42 parts, among them U16 AP61202Z6, U18 AP61202Z6, U19 AP61202Z6, U6 NCP163ASN330T1G, U8 AP61202Z6

Commit message: Schematic reorg step 9: ERC to zero
- Wires trimmed back to their last label or cap (SDM config lines, LPDDR4
  decoupling rows, PG pins); loose stubs and R29 leftovers removed
- Unused bus links removed: {iob6a}, {iobank_2aB}, {iob6c}, {phy} and the
  io_headers {jtag} (sheet pins, root buses, unnamed internal buses);
  {iob6b} bus tail trimmed

Netdiff: 0 renamed, 0 connectivity diffs. ERC 21 -> 0. PCB unchanged, DRC parity 0.
Changed lines of the file:
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@@
-	)
-	(junction
-		(at 58.42 91.44)
-		(diameter 0)
-		(color 0 0 0 0)
 	)
 	(junction
@@
 	(wire
 		(pts
-			(xy 58.42 91.44) (xy 63.5 91.44)
-		)
-		(stroke
-			(width 0)
-			(type default)
-		)
-	)
-	(wire
-		(pts
 			(xy 130.81 133.35) (xy 133.35 133.35)
 		)
@@
 	(wire
 		(pts
-			(xy 102.87 119.38) (xy 107.95 119.38)
+			(xy 102.87 119.38) (xy 104.14 119.38)
 		)
 		(stroke
@@
 	(wire
 		(pts
-			(xy 102.87 24.13) (xy 107.95 24.13)
+			(xy 102.87 24.13) (xy 104.14 24.13)
 		)
 		(stroke
@@
 	(wire
 		(pts
-			(xy 102.87 87.63) (xy 107.95 87.63)
-		)
-		(stroke
+			(xy 102.87 87.63) (xy 104.14 87.63)
+		)
+		(stroke
