File: a5e_kicad/pwr_vcore.kicad_sch (KiCad schematic)
At the start: 27 parts, among them U15 TPS548A28RWWR

Commit message: Schematic reorg step 9: ERC to zero
- Wires trimmed back to their last label or cap (SDM config lines, LPDDR4
  decoupling rows, PG pins); loose stubs and R29 leftovers removed
- Unused bus links removed: {iob6a}, {iobank_2aB}, {iob6c}, {phy} and the
  io_headers {jtag} (sheet pins, root buses, unnamed internal buses);
  {iob6b} bus tail trimmed

Netdiff: 0 renamed, 0 connectivity diffs. ERC 21 -> 0. PCB unchanged, DRC parity 0.
Changed lines of the file:
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@@
-	(wire
-		(pts
-			(xy 123.19 181.61) (xy 123.19 184.15)
-		)
-		(stroke
-			(width 0)
-			(type default)
-		)
-	)
 	(wire
 		(pts
@@
 		(pts
 			(xy 128.27 137.16) (xy 148.59 137.16)
-		)
-		(stroke
-			(width 0)
-			(type default)
-		)
-	)
-	(wire
-		(pts
-			(xy 123.19 184.15) (xy 115.57 184.15)
 		)
 		(stroke
@@
 		)
 		(stroke
-			(width 0)
-			(type default)
-		)
-	)
-	(wire
-		(pts
-			(xy 123.19 173.99) (xy 123.19 171.45)
-		)
-		(stroke
