File: agilex_3_soc.kicad_pcb (KiCad board)
At the start: 8 copper layers, 76 x 65.1 mm, 305 parts, among them J1 Conn_01x05, J10 HPS_UART_3V3, J2 Conn_01x03, J3 Conn_02x19_Odd_Even, J4 Conn_01x03, J5 Conn_01x14, J6 Conn_02x03_Odd_Even, J8 Micro_SD_Card, J9 RJ45_RB1-125B8G1A, U1 SN74AXC4T774PWR, U10 KSZ9031RNXCA, U11 NXS0506GUX, U12 IS43LQ32256A-062BLI, U15 TDA38812XUMA1, U16 AP61202Z6, U18 AP61202Z6, U19 AP61202Z6, U2 MX25U25645G, U3 CD4051B, U4 AD8603, U40 TPS2116DRLR, U41 TPS22918DBVR, U42 SN74AXC4T774PWR, U5 ADS7056IRUGR, U6 NCP163ASN330T1G, U7 A5EB013B-B23B, U8 AP61202Z6, U9 AX3HAF1-100.0000, Y2 SIT8924BA-73-18N-25.000000, Y3 25MHz

Commit message: Remove leftover 1V8 stub from R247 pad 2
R247 (PHY RESET_N pull-up) was changed from 1V8 to pg_all in 480705d but
the old B.Cu 1V8 track to the pad remained, shorting pg_all to 1V8. Also
remove the 1V8 via it ended on and its F.Cu tail, which were redundant.
R247 pad 2 now shows a pg_all ratsnest to be routed.
Routing:
- net 1V8: track 110.3 -> 109.0 mm, vias 52 -> 51
Changed lines of the file:
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@@
-	)
-	(segment
-		(start 182.50184 102.53415)
-		(end 183.09184 102.53415)
-		(width 0.1)
-		(layer "F.Cu")
-		(net "1V8")
 	)
 	(segment
@@
 	)
 	(segment
-		(start 183.09184 102.53415)
-		(end 183.11684 102.50915)
-		(width 0.1)
-		(layer "F.Cu")
-		(net "1V8")
-	)
-	(segment
 		(start 178.49184 107.58415)
 		(end 177.94184 107.58415)
@@
 	(via
 		(at 185.56684 115.00915)
-		(size 0.3)
-		(drill 0.15)
-		(layers "F.Cu" "B.Cu")
-		(net "1V8")
-	)
-	(via
-		(at 183.11684 102.50915)
 		(size 0.3)
 		(drill 0.15)
@@
 	)
 	(segment
-		(start 182.48684 102.23415)
-		(end 182.84184 102.23415)
-		(width 0.1)
-		(layer "B.Cu")
-		(net "1V8")
-	)
-	(segment
 		(start 178.84184 111.23415)
 		(end 178.84184 111.79415)
@@
 		(width 0.1)
 		(layer "B.Cu")
-		(net "1V8")
-	)
-	(segment
-		(start 182.84184 102.23415)
-		(end 183.11684 102.50915)
-		(width 0.1)
-		(layer "B.Cu")
