File: agilex_3_soc.kicad_pcb (KiCad board)
At the start: 8 copper layers, 76 x 65.1 mm, 314 parts, among them J1 Conn_01x05, J10 HPS_UART_3V3, J2 Conn_01x03, J3 2x19 1.27mm socket, bottom, J4 Conn_01x03, J5 Conn_01x14, J6 Conn_02x03_Odd_Even, J8 Micro_SD_Card, J9 RJ45_RB1-125B8G1A, U1 SN74AXC4T774PWR, U10 KSZ9031RNXCA, U11 NXS0506GUX, U12 H9HCNNN8KUMLHR-NME, U15 TDA38812XUMA1, U16 AP61202Z6, U18 AP61202Z6, U19 AP61202Z6, U2 IS25WP128-RHLE, U3 CD4051B, U4 AD8603, U40 TPS2116DRLR, U41 TPS22918DBVR, U42 SN74AXC4T774PWR, U5 ADS7056IRUGR, U6 NCP163ASN330T1G, U7 A5EB013B-B23B, U8 AP61202Z6, U9 AX3HAF1-100.0000, Y2 SIT8924BA-73-18N-25.000000, Y3 25MHz

Commit message: PCB: add fiducials, three per side
1 mm copper / 2 mm mask fiducials in asymmetric patterns: top FID1-3,
bottom FID4-6, each >= 3 mm from the edge and clear of copper and
courtyards. They are board-only, excluded from the BOM and the position
file.
Parts:
- added FID1: Fiducial, Fiducial:Fiducial_1mm_Mask2mm, F.Cu at (132.8, 85.9)
- added FID2: Fiducial, Fiducial:Fiducial_1mm_Mask2mm, F.Cu at (127.0, 145.0)
- added FID3: Fiducial, Fiducial:Fiducial_1mm_Mask2mm, F.Cu at (190.5, 145.0)
- added FID4: Fiducial, Fiducial:Fiducial_1mm_Mask2mm, B.Cu at (195.3, 89.9)
- added FID5: Fiducial, Fiducial:Fiducial_1mm_Mask2mm, B.Cu at (127.0, 145.0)
- added FID6: Fiducial, Fiducial:Fiducial_1mm_Mask2mm, B.Cu at (197.0, 139.3)
